File: sensing_audio_visual_PCB.kicad_sch (KiCad schematic)
At the start: 9 parts, among them J1 Amplifier, J2 OLED Display, J3 IR Emitter, J4 Light Strip, J5 Conn_01x03, J6 IR Receiver, J7 220 ohm, J8 10k ohm, J9 OLED Display

Commit message: KiCad schemitc
Parts:
- added J10, J14, J18: 220 ohm, symbol Connector_Generic:Conn_01x02
- added J11, J15, J20: IR Emitter, symbol Connector_Generic:Conn_01x02
- added J12, J16, J19: 10k ohm, symbol Connector_Generic:Conn_01x02
- added J13, J17, J21: IR Receiver, symbol Connector_Generic:Conn_01x02
Connections:
- net 5V is gone; now on net 3V3: J3.2 (Pin_2), J4.1 (Pin_1), J5.1 (Pin_1)
- net 3V3: now also J10.1 (Pin_1), J11.2 (Pin_2), J12.1 (Pin_1), J14.1 (Pin_1), J15.2 (Pin_2), J16.1 (Pin_1), J18.1 (Pin_1), J19.1 (Pin_1), J20.2 (Pin_2)
- net GND: now also J13.2 (Pin_2), J17.2 (Pin_2), J21.2 (Pin_2)
- new net: J14.2 (Pin_2), J15.1 (Pin_1)
- new net: J18.2 (Pin_2), J20.1 (Pin_1)
- new net: J19.2 (Pin_2), J21.1 (Pin_1)
- new net: J12.2 (Pin_2), J13.1 (Pin_1)
- new net: J16.2 (Pin_2), J17.1 (Pin_1)
- new net: J10.2 (Pin_2), J11.1 (Pin_1)
Other:
- moved on the sheet: J3, J6, J7, J8, J9

Commit message: Footprints added
Parts:
- J1, J4, J5: footprint (none) -> Connector_PinHeader_2.54mm:PinHeader_1x03_P2.54mm_Vertical
- J10, J12, J14, J16, J18, J19, J7, J8: footprint (none) -> Resistor_THT:R_Axial_DIN0207_L6.3mm_D2.5mm_P7.62mm_Horizontal
- J11, J13, J17, J20, J21, J3, J6: footprint (none) -> TestPoint:TestPoint_2Pads_Pitch5.08mm_Drill1.3mm
- J15: footprint (none) -> TestPoint_2Pads_Pitch5.08mm_Drill1.3mm
- J2: footprint (none) -> Connector_PinHeader_2.54mm:PinHeader_1x04_P2.54mm_Vertical
- J9: value OLED Display -> GPIO Pins; footprint (none) -> Connector_PinHeader_2.54mm:PinHeader_1x04_P2.54mm_Vertical
Connections:
- net 3V3: no longer J10.1 (Pin_1), J11.2 (Pin_2), J14.1 (Pin_1), J15.2 (Pin_2), J18.1 (Pin_1), J20.2 (Pin_2), J3.2 (Pin_2), J4.1 (Pin_1), J4.2 (Pin_2), J5.1 (Pin_1), J7.1 (Pin_1)
- net GND: now also J11.2 (Pin_2), J15.2 (Pin_2), J20.2 (Pin_2), J3.2 (Pin_2)
- net at J19.2 (Pin_2), J21.1 (Pin_1): now also J9.2 (Pin_2)
- net at J12.2 (Pin_2), J13.1 (Pin_1): now also J9.4 (Pin_4)
- net at J9.1 (Pin_1): now also J16.2 (Pin_2), J17.1 (Pin_1)
- net at J9.3 (Pin_3): now also J6.1 (Pin_1), J8.2 (Pin_2)
- new net 5V: J10.1 (Pin_1), J14.1 (Pin_1), J18.1 (Pin_1), J4.1 (Pin_1), J5.1 (Pin_1), J7.1 (Pin_1)
- new net DIN: J4.2 (Pin_2)
Other:
- moved on the sheet: J9

Commit message: Layout finished
Parts:
- removed J9: GPIO Pins, Connector_PinHeader_2.54mm:PinHeader_1x04_P2.54mm_Vertical, symbol Connector_Generic:Conn_01x04
- added J22, J25: R_PhotoR, Resistor_THT:R_Axial_DIN0207_L6.3mm_D2.5mm_P7.62mm_Horizontal, symbol Connector_Generic:Conn_01x02
- added J23, J26: photoresistor, TestPoint:TestPoint_2Pads_Pitch5.08mm_Drill1.3mm, symbol Connector_Generic:Conn_01x02
- added J27, J29: R_LED, Resistor_THT:R_Axial_DIN0207_L6.3mm_D2.5mm_P7.62mm_Horizontal, symbol Connector_Generic:Conn_01x02
- added J28, J30: LED, TestPoint:TestPoint_2Pads_Pitch5.08mm_Drill1.3mm, symbol Connector_Generic:Conn_01x02
- added J9: Conn_01x06, Connector_PinHeader_2.54mm:PinHeader_1x06_P2.54mm_Vertical, symbol Connector_Generic:Conn_01x06
- J10, J14, J18, J7: value 220 ohm -> R_emitter
- J12, J16, J19, J8: value 10k ohm -> R_receiver
Connections:
- net 3V3: now also J22.1 (Pin_1), J25.1 (Pin_1), J27.1 (Pin_1), J29.1 (Pin_1)
- net GND: now also J23.2 (Pin_2), J26.2 (Pin_2), J28.2 (Pin_2), J30.2 (Pin_2)
- net at J19.2 (Pin_2), J21.1 (Pin_1): now also J9.2 (Pin_2)
- net at J12.2 (Pin_2), J13.1 (Pin_1): now also J9.4 (Pin_4)
- net at J16.2 (Pin_2), J17.1 (Pin_1): now also J9.1 (Pin_1)
- net at J6.1 (Pin_1), J8.2 (Pin_2): now also J9.3 (Pin_3)
- new net: J25.2 (Pin_2), J26.1 (Pin_1), J9.6 (Pin_6)
- new net: J22.2 (Pin_2), J23.1 (Pin_1), J9.5 (Pin_5)
- new net: J29.2 (Pin_2), J30.1 (Pin_1)
- new net: J27.2 (Pin_2), J28.1 (Pin_1)
Other:
- moved on the sheet: J1, J10, J11, J12, J13, J14, J15, J16, J17, J18, J19, J2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
